File: ESP32-S3-WROOM-1U.kicad_sch (KiCad schematic)
At the start: 24 parts, among them U201 ESP32-S3-WROOM-1U-N16R8

Commit message: Updated symbols, added jobset and output folders.
Parts:
- C201: Manufacturer (none) -> Samsung Electro-Mechanics; Manufacturer Part No (none) -> CL21B105KBFNNNE
- C202: Manufacturer (none) -> Samsung Electro-Mechanics; Manufacturer Part No (none) -> CL31A106KBHNNNE
- R207, R208: Manufacturer (none) -> UNI-ROYAL(Uniroyal Elec); Manufacturer Part No (none) -> 0805W8F220JT5E
- R209, R210: Manufacturer (none) -> UNI-ROYAL(Uniroyal Elec); Manufacturer Part No (none) -> 0805W8F4701T5E
- R211, R212, R213: Manufacturer (none) -> UNI-ROYAL(Uniroyal Elec); Manufacturer Part No (none) -> 0805W8F470JT5E
Changed lines of the file:
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@@
 	)
 	(symbol
-		(lib_name "0805W8F1002T5E_2")
 		(lib_id "JLCPCB Basic:0805W8F1002T5E")
 		(at 195.58 114.3 0)
@@
 			)
 		)
+		(property "Manufacturer" "UNI-ROYAL(Uniroyal Elec)"
+			(at 250.19 -566.65 0)
+			(effects
+				(font
+					(size 1.27 1.27)
+				)
+				(justify left top)
+				(hide yes)
+			)
+		)
+		(property "Manufacturer Part No" "0805W8F470JT5E"
+			(at 250.19 -666.65 0)
+			(effects
+				(font
+					(size 1.27 1.27)
+				)
+				(justify left top)
+				(hide yes)
+			)
+		)
 		(pin "1"
 		)
@@
 	)
 	(symbol
-		(lib_name "CC0603KRX7R9BB104_1")
 		(lib_id "JLCPCB Basic:CC0603KRX7R9BB104")
 		(at 144.78 152.4 0)
@@
 	)
 	(symbol
-		(lib_name "0805W8F1002T5E_2")
 		(lib_id "JLCPCB Basic:0805W8F1002T5E")
 		(at 195.58 142.24 0)
@@
 	)
 	(symbol
-		(lib_name "CC0603KRX7R9BB104_1")
 		(lib_id "JLCPCB Basic:CC0603KRX7R9BB104")
 		(at 97.79 152.4 0)
@@
 	)
 	(symbol
-		(lib_name "0805W8F4701T5E_1")
 		(lib_id "JLCPCB Basic:0805W8F4701T5E")
 		(at 233.68 40.64 0)
@@
 			)
 		)
+		(property "Manufacturer" "UNI-ROYAL(Uniroyal Elec)"
+			(at 247.65 736.83 0)
+			(effects
+				(font
+					(size 1.27 1.27)
+				)
+				(justify left top)
+				(hide yes)
+			)
+		)
+		(property "Manufacturer Part No" "0805W8F4701T5E"
+			(at 247.65 836.83 0)
+			(effects
+				(font
+					(size 1.27 1.27)
+				)
+				(justify left top)
+				(hide yes)
+			)
+		)
 		(pin "1"
 		)
@@
 			)
 		)
+		(property "Manufacturer" "UNI-ROYAL(Uniroyal Elec)"
+			(at 229.87 774.93 0)
+			(effects
+				(font
+					(size 1.27 1.27)
+				)
+				(justify left top)
+				(hide yes)
+			)
+		)
+		(property "Manufacturer Part No" "0805W8F220JT5E"
+			(at 229.87 874.93 0)
+			(effects
+				(font
+					(size 1.27 1.27)
+				)
+				(justify left top)
+				(hide yes)
+			)
+		)
 		(pin "1"
 		)
@@
 	)
 	(symbol
-		(lib_name "0805W8F1002T5E_2")
 		(lib_id "JLCPCB Basic:0805W8F1002T5E")
 		(at 195.58 124.46 0)
@@
 			)
 		)
+		(property "Manufacturer" "UNI-ROYAL(Uniroyal Elec)"
+			(at 250.19 -574.27 0)
+			(effects
+				(font
+					(size 1.27 1.27)
+				)
+				(justify left top)
+				(hide yes)
+			)
+		)
+		(property "Manufacturer Part No" "0805W8F470JT5E"
+			(at 250.19 -674.27 0)
+			(effects
+				(font
+					(size 1.27 1.27)
+				)
+				(justify left top)
+				(hide yes)
+			)
+		)
 		(pin "1"
 		)
@@
 			)
 		)
+		(property "Manufacturer" "UNI-ROYAL(Uniroyal Elec)"
+			(at 250.19 -559.03 0)
+			(effects
+				(font
+					(size 1.27 1.27)
+				)
+				(justify left top)
+				(hide yes)
+			)
+		)
+		(property "Manufacturer Part No" "0805W8F470JT5E"
+			(at 250.19 -659.03 0)
+			(effects
+				(font
+					(size 1.27 1.27)
+				)
+				(justify left top)
+				(hide yes)
+			)
+		)
 		(pin "1"
 		)
@@
 			)
 		)
+		(property "Manufacturer" "UNI-ROYAL(Uniroyal Elec)"
+			(at 229.87 778.74 0)
+			(effects
+				(font
+					(size 1.27 1.27)
+				)
+				(justify left top)
+				(hide yes)
+			)
+		)
+		(property "Manufacturer Part No" "0805W8F220JT5E"
+			(at 229.87 878.74 0)
+			(effects
+				(font
+					(size 1.27 1.27)
+				)
+				(justify left top)
+				(hide yes)
+			)
+		)
 		(pin "1"
 		)
@@
 			)
 		)
+		(property "Manufacturer" "Samsung Electro-Mechanics"
+			(at 83.82 -655.55 0)
+			(effects
+				(font
+					(size 1.27 1.27)
+				)
+				(justify left top)
+				(hide yes)
+			)
+		)
+		(property "Manufacturer Part No" "CL31A106KBHNNNE"
+			(at 83.82 -755.55 0)
+			(effects
+				(font
+					(size 1.27 1.27)
+				)
+				(justify left top)
+				(hide yes)
+			)
+		)
 		(pin "2"
 		)
@@
 	)
 	(symbol
-		(lib_name "0805W8F1002T5E_2")
 		(lib_id "JLCPCB Basic:0805W8F1002T5E")
 		(at 195.58 132.08 0)
@@
 			)
 		)
+		(property "Manufacturer" "Samsung Electro-Mechanics"
+			(at 76.2 -543.79 0)
+			(effects
+				(font
+					(size 1.27 1.27)
+				)
+				(justify left top)
+				(hide yes)
+			)
+		)
+		(property "Manufacturer Part No" "CL21B105KBFNNNE"
+			(at 76.2 -643.79 0)
+			(effects
+				(font
+					(size 1.27 1.27)
+				)
+				(justify left top)
+				(hide yes)
+			)
+		)
 		(pin "1"
 		)
@@
 	)
 	(symbol
-		(lib_name "0805W8F4701T5E_1")
 		(lib_id "JLCPCB Basic:0805W8F4701T5E")
 		(at 233.68 33.02 0)
@@
 				(hide yes)
 			)
+		)
+		(property "Manufacturer" "UNI-ROYAL(Uniroyal Elec)"
+			(at 247.65 729.21 0)
+			(effects
+				(font
+					(size 1.27 1.27)
+				)
+				(justify left top)
+				(hide yes)
+			)
+		)
+		(property "Manufacturer Part No" "0805W8F4701T5E"
+			(at 247.65 829.21 0)
+			(effects
+				(font
+					(size 1.27 1.27)
+				)
+				(justify left top)
+				(hide yes)
+			)

Commit message: Updated inductor component and 10uF capacitor components to bring down cost.
Parts:
- removed C202: 10uF 10% 50V, JLCPCB Basic:CAPC3216X180N, symbol JLCPCB Basic:CL31A106KBHNNNE
- added C201: 10uF 10% 25V, JLCPCB Basic:CAPC3216X180N, symbol SAMSUNGELECTROMECHANICS Resistors:CL31A106KAHNNNE
- renumbered C201 to C202
Connections:
- net +3V3: now also C201.2
- net GND: now also C201.1
Changed lines of the file:
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@@
 	)
 	(symbol
+		(lib_id "SAMSUNGELECTROMECHANICS Resistors:CL31A106KAHNNNE")
+		(at 85.09 40.64 0)
+		(unit 1)
+		(exclude_from_sim no)
+		(in_bom yes)
+		(on_board yes)
+		(dnp no)
+		(fields_autoplaced yes)
+		(property "Reference" "C201"
+			(at 88.9 33.02 0)
+			(effects
+				(font
+					(size 1.27 1.27)
+				)
+			)
+		)
+		(property "Value" "10uF 10% 25V"
+			(at 88.9 35.56 0)
+			(effects
+				(font
+					(size 1.27 1.27)
+				)
+			)
+		)
+		(property "Footprint" "JLCPCB Basic:CAPC3216X180N"
+			(at 93.98 136.83 0)
+			(effects
+				(font
+					(size 1.27 1.27)
+				)
+				(justify left top)
+				(hide yes)
+			)
+		)
+		(property "Datasheet" ""
+			(at 93.98 236.83 0)
+			(effects
+				(font
+					(size 1.27 1.27)
+				)
+				(justify left top)
+				(hide yes)
+			)
+		)
+		(property "Description" "Capacitor Ceramic, 10uF, 25V, 1206, 10%, X5R"
+			(at 88.9 45.72 0)
+			(effects
+				(font
+					(size 1.27 1.27)
+				)
+				(hide yes)
+			)
+		)
+		(property "Height" "1.8"
+			(at 93.98 436.83 0)
+			(effects
+				(font
+					(size 1.27 1.27)
+				)
+				(justify left top)
+				(hide yes)
+			)
+		)
+		(property "Manufacturer" "Samsung Electro-Mechanics"
+			(at 93.98 736.83 0)
+			(effects
+				(font
+					(size 1.27 1.27)
+				)
+				(justify left top)
+				(hide yes)
+			)
+		)
+		(property "Manufacturer Part No" "CL31A106KAHNNNE"
+			(at 93.98 836.83 0)
+			(effects
+				(font
+					(size 1.27 1.27)
+				)
+				(justify left top)
+				(hide yes)
+			)
+		)
+		(property "JLCPCB Part #" "C9807"
+			(at 89.154 48.006 0)
+			(effects
+				(font
+					(size 1.27 1.27)
+				)
+				(hide yes)
+			)
+		)
+		(property "Package" "1206"
+			(at 89.408 50.038 0)
+			(effects
+				(font
+					(size 1.27 1.27)
+				)
+				(hide yes)
+			)
+		)
+		(property "Part Type" "Basic"
+			(at 89.408 52.07 0)
+			(effects
+				(font
+					(size 1.27 1.27)
+				)
+				(hide yes)
+			)
+		)
+		(pin "1"
+		)
+		(pin "2"
+		)
+		(instances
+			(project ""
+				(path "/fb66fec7-a625-41b0-8b4b-639a0ec63be1/688027c4-6d3d-464d-b364-684d75515e96"
+					(reference "C201")
+					(unit 1)
+				)
+			)
+		)
+	)
+	(symbol
 		(lib_id "JLCPCB Basic:CC0603KRX7R9BB104")
 		(at 97.79 152.4 0)
@@
 	)
 	(symbol
-		(lib_id "JLCPCB Basic:CL31A106KBHNNNE")
-		(at 92.71 40.64 180)
-		(unit 1)
-		(exclude_from_sim no)
-		(in_bom yes)
-		(on_board yes)
-		(dnp no)
-		(property "Reference" "C202"
-			(at 86.106 34.036 0)
-			(effects
-				(font
-					(size 1.27 1.27)
-				)
-				(justify right)
-			)
-		)
-		(property "Value" "10uF 10% 50V"
-			(at 82.042 36.322 0)
-			(effects
-				(font
-					(size 1.27 1.27)
-				)
-				(justify right)
-			)
-		)
-		(property "Footprint" "JLCPCB Basic:CAPC3216X180N"
-			(at 83.82 -55.55 0)
-			(effects
-				(font
-					(size 1.27 1.27)
-				)
-				(justify left top)
-				(hide yes)
-			)
-		)
-		(property "Datasheet" "https://datasheet.datasheetarchive.com/originals/distributors/Datasheets_SAMA/08745f6325ae1679773301b11fb0567f.pdf"
-			(at 83.82 -155.55 0)
-			(effects
-				(font
-					(size 1.27 1.27)
-				)
-				(justify left top)
-				(hide yes)
-			)
-		)
-		(property "Description" "Capacitor Ceramic, 10uF, 50V, 1206, 10%, X5R"
-			(at 88.9 35.56 0)
-			(effects
-				(font
-					(size 1.27 1.27)
-				)
-				(hide yes)
-			)
-		)
-		(property "Height" "1.8"
-			(at 83.82 -355.55 0)
-			(effects
-				(font
-					(size 1.27 1.27)
-				)
-				(justify left top)
-				(hide yes)
-			)
-		)
-		(property "Mouser Part Number" "187-CL31A106KBHNNNE"
-			(at 83.82 -455.55 0)
-			(effects
-				(font
-					(size 1.27 1.27)
-				)
-				(justify left top)
-				(hide yes)
-			)
-		)
-		(property "Mouser Price/Stock" "https://au.mouser.com/ProductDetail/Samsung-Electro-Mechanics/CL31A106KBHNNNE?qs=X6jEic%2FHinBsSMnC%2FFnmbg%3D%3D"
-			(at 83.82 -555.55 0)
-			(effects
-				(font
-					(size 1.27 1.27)
-				)
-				(justify left top)
-				(hide yes)
-			)
-		)
-		(property "Manufacturer_Name" "Samsung Electro-Mechanics"
-			(at 83.82 -655.55 0)
-			(effects
-				(font
-					(size 1.27 1.27)
-				)
-				(justify left top)
-				(hide yes)
-			)
-		)
-		(property "Manufacturer_Part_Number" "CL31A106KBHNNNE"
-			(at 83.82 -755.55 0)
-			(effects
-				(font
-					(size 1.27 1.27)
-				)
-				(justify left top)
-				(hide yes)
-			)
-		)
-		(property "JLCPCB Part #" "C13585"
-			(at 88.646 33.274 0)
-			(effects
-				(font
-					(size 1.27 1.27)
-				)
-				(hide yes)
-			)
-		)
-		(property "Package" "1206"
-			(at 88.392 31.242 0)
-			(effects
-				(font
-					(size 1.27 1.27)
-				)
-				(hide yes)
-			)
-		)
-		(property "Part Type" "Basic"
-			(at 88.392 29.21 0)
-			(effects
-				(font
-					(size 1.27 1.27)
-				)
-				(hide yes)
-			)
-		)
-		(property "PCB_Hint" "Decoupling, close as possible to ESP32"
-			(at 92.71 40.64 0)
-			(effects
-				(font
-					(size 1.27 1.27)
-				)
-				(hide yes)
-			)
-		)
-		(property "Manufacturer" "Samsung Electro-Mechanics"
-			(at 83.82 -655.55 0)
-			(effects
-				(font
-					(size 1.27 1.27)
-				)
-				(justify left top)
-				(hide yes)
-			)
-		)
-		(property "Manufacturer Part No" "CL31A106KBHNNNE"
-			(at 83.82 -755.55 0)
-			(effects
-				(font
-					(size 1.27 1.27)
-				)
-				(justify left top)
-				(hide yes)
-			)
-		)
-		(pin "2"
-		)
-		(pin "1"
-		)
-		(instances
-			(project "MQTT-ModularControllerBoard"
-				(path "/fb66fec7-a625-41b0-8b4b-639a0ec63be1/688027c4-6d3d-464d-b364-684d75515e96"
-					(reference "C202")
-					(unit 1)
-				)
-			)
-		)
-	)
-	(symbol
 		(lib_id "JLCPCB Basic:0805W8F1002T5E")
 		(at 195.58 132.08 0)
@@
 		(on_board yes)
 		(dnp no)
-		(property "Reference" "C201"
+		(property "Reference" "C202"
 			(at 78.232 146.05 0)
 			(effects
@@
 			(project ""
 				(path "/fb66fec7-a625-41b0-8b4b-639a0ec63be1/688027c4-6d3d-464d-b364-684d75515e96"
-					(reference "C201")
+					(reference "C202")
 					(unit 1)
 				)

Commit message: Updated Fab layer and silkscreen.
Parts:
- U201: footprint PCM_Espressif:ESP32-S3-WROOM-1U -> ESPRESSIF Microcontrollers:ESP32-S3-WROOM-1U
Changed lines of the file:
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@@
 			)
 		)
-		(property "Footprint" "PCM_Espressif:ESP32-S3-WROOM-1U"
+		(property "Footprint" "ESPRESSIF Microcontrollers:ESP32-S3-WROOM-1U"
 			(at 99.06 143.002 0)
 			(effects
